File: RemiRAT.kicad_pcb (KiCad board)
At the start: 4 copper layers, 73 x 57 mm, 49 parts, among them J3 PinHeader_1x06_P2.54mm_Vertic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, J6 PinHeader_1x06_P2.54mm_Vertic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, J7 PinHeader_1x04_P2.54mm_Vertic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, J8 PinHeader_2x06_P2.54mm_Vertic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, J9 ESP BREAKOUT, Y1 12MHz 13pF 60Ohms, Y2 32.768 kHz 7 pF 70 kOhms

Commit message: Add files via upload
Parts:
- removed the REF** at (139.5, 100.5)
- removed the REF** at (133.5, 99.5)
- added C11: 220uF 50V, Capacitor_THT:CP_Radial_D10.0mm_P5.00mm, F.Cu at (173.6, 103.5)
- added C12: 1uF 50V, Capacitor_SMD:C_0805_2012Metric, F.Cu at (169.0, 102.5)
- added C13: 47uF 25V, Capacitor_SMD:C_1206_3216Metric, F.Cu at (161.0, 118.0)
- added C14: 1uF 25V, Capacitor_SMD:C_0402_1005Metric, F.Cu at (146.0, 117.0)
- added C15: 25V 0.1uF, Capacitor_SMD:C_0402_1005Metric, F.Cu at (140.0, 100.0)
- added C16: 25V 10uF, Capacitor_SMD:C_0805_2012Metric, F.Cu at (140.5, 101.5)
- added C17: 25V 0.1uF, Capacitor_SMD:C_0402_1005Metric, F.Cu at (143.0, 100.5)
- added C18: 25V 0.1uF, Capacitor_SMD:C_0402_1005Metric, F.Cu at (134.0, 100.0)
- added C19: 25V 0.1uF, Capacitor_SMD:C_0402_1005Metric, F.Cu at (125.0, 83.0)
- added C20: 25V 0.1uF, Capacitor_SMD:C_0402_1005Metric, F.Cu at (139.0, 74.5)
- added C21: 25V 0.1uF, Capacitor_SMD:C_0402_1005Metric, F.Cu at (150.5, 80.0)
- added F1: 1.5A 32V SLOWBLOW, Fuse:Fuse_0603_1608Metric_Pad1.05x0.95mm_HandSolder, F.Cu at (124.5, 111.0)
- added F3: 2A 32V SlowBlow, Fuse:Fuse_0603_1608Metric_Pad1.05x0.95mm_HandSolder, F.Cu at (180.5, 110.0)
- added J10: , TerminalBlock_TE-Connectivity:TerminalBlock_TE_282834-2_1x02_P2.54mm_Horizontal, F.Cu at (177.0, 116.4)
- added J11: PinHeader_1x03_P2.54mm_Vertical, Connector_PinHeader_2.54mm:PinHeader_1x03_P2.54mm_Vertical, F.Cu at (136.0, 117.0)
- added R13: 4.7K Ohm, Resistor_SMD:R_0402_1005Metric, F.Cu at (146.0, 100.5)
- added R14: 4.7K Ohm, Resistor_SMD:R_0402_1005Metric, F.Cu at (125.5, 82.0)
- added REF**: NetTie-3_SMD_Pad0.5mm, NetTie:NetTie-3_SMD_Pad0.5mm, F.Cu at (139.0, 95.5)
- added VR2: CONV_TSR_2-2450, TSR_2_2450:CONV_TSR_2-2450, F.Cu at (166.9, 113.0)
- F2: value 1.5A 32V -> 1.5A 32V FASTBLOW
- moved J4 55.2 mm to (150.5, 60.5), turned to 180 degrees
- moved J7 41.5 mm to (140.0, 56.7), turned to 0 degrees
- moved S3 26.0 mm to (129.0, 64.0), turned to 90 degrees
- moved S1 22.9 mm to (156.4, 94.6), turned to 180 degrees
- moved J9 22.0 mm to (182.7, 77.7)
- moved J6 21.0 mm to (135.0, 56.4), turned to 0 degrees
- moved C2 20.4 mm to (121.0, 109.5), turned to 180 degrees
- moved C1 17.0 mm to (121.5, 111.0), turned to 180 degrees
- moved J2 16.1 mm to (175.2, 78.0)
- moved U2 15.8 mm to (173.6, 62.3)
- moved C8 15.7 mm to (160.5, 57.0)
- moved C9 15.7 mm to (162.5, 56.0)
- moved F4 13.9 mm to (148.5, 115.5)
- moved J3 13.5 mm to (188.0, 59.5)
- moved R10 11.3 mm to (165.6, 82.5), turned to 90 degrees
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- renumbered F1 to F4
Connections:
- F4 pad 1: VBUS -> 3.3V
- F4 pad 2: VBUS -> 3.3V
- S1 pad 1: NRSTB -> EN
- U1 pad 46: SAM_JTAGSEL_PIN46 -> GND
Routing:
- net SAM-SPI-NPCS0: track 50.9 -> 9.37 mm, vias 2 -> 0
- net GND: track 95.9 -> 132.7 mm, vias 7 -> 21
- net VIN: track 0.00 -> 29.4 mm
- net VDDCORE: track 55.4 -> 83.5 mm, vias 6 -> 8
- net SAM-SPI-MOSI: track 47.8 -> 21.2 mm, vias 1 -> 0
- net VBUS: track 54.8 -> 80.4 mm, vias 7 -> 5
- net TWD0/PA17: track 13.1 -> 33.5 mm
- net IO26: track 70.1 -> 51.3 mm
- net VDDPLL: track 2.19 -> 20.3 mm, vias 0 -> 2
- net NRSTB: track 101.6 -> 84.2 mm, vias 3 -> 5
- net SAM-SPI-SCK: track 45.4 -> 28.8 mm, vias 1 -> 0
- net CANRX0/PA1: track 23.0 -> 39.0 mm
- net CANTX0/PA0: track 21.4 -> 37.3 mm
- net 3.3V: track 38.0 -> 52.5 mm, vias 13 -> 16
- net TWCK0/PA18: track 39.0 -> 53.5 mm
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Other:
- board size 73 x 57 mm -> 73 x 69.5 mm
- board text added: "1 3 5 7"
- board text added: "11 9 7 5 3 1"
- board text added: "12 10 8 6 4 2"
- board text added: "1:IO17 2:IO5 3:IO16 4:IO18 5:IO4 6:IO19 7:IO2 8:IO21"
- board text added: "1=SAM-RST 2=ESP-FLASH 3&4=NC"
- board text added: "2 4 6 8"
- board text added: "6.5V-24V"
- board text added: "ESP BREAKOUT"
- board text added: "RST"
- board text added: "SAM BREAKOUT"
- board text added: "SAM SPI1"
- board text added: "USBC"
- board text added: "VIN"
- board text removed: "1 3 5 7 9 11"
- board text removed: "1 = SAM-RST 2 = ESP-FLASH 3 = NC 4 = NC"
- board text removed: "1:IO17 3:IO16 5:IO4 7:IO2"
- board text removed: "2 4 6 8 10 12"
- board text removed: "IO5:2 IO18:4 IO19:6 IO21:8"
- board text removed: "SAM RST"
- board text removed: "SAMSPI1"
