File: RemiRAT.kicad_pcb (KiCad board)
At the start: 4 copper layers, 73 x 69.5 mm, 73 parts, among them J11 PinHeader_1x03_P2.54mm_Vertic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, J3 PinHeader_1x06_P2.54mm_Vertic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, J6 PinHeader_1x06_P2.54mm_Vertic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, J7 PinHeader_1x04_P2.54mm_Vertic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, J8 PinHeader_2x06_P2.54mm_Vertic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, J9 ESP BREAKOUT, Y1 12MHz 13pF 60Ohms, Y2 32.768 kHz 7 pF 70 kOhms

Commit message: Add files via upload
Parts:
- added C25: 25V 0.1uF, Capacitor_SMD:C_0402_1005Metric, F.Cu at (181.5, 91.0)
- added F5: 1.5A 32V FastBlow, Fuse:Fuse_0402_1005Metric_Pad0.77x0.64mm_HandSolder, F.Cu at (155.6, 118.0)
- added J12: , Connector_PinHeader_2.54mm:PinHeader_1x03_P2.54mm_Vertical, F.Cu at (187.0, 98.4)
- added J14: , Connector_PinHeader_2.54mm:PinHeader_1x02_P2.54mm_Vertical, F.Cu at (154.8, 115.5)
- added J15: BarrelJack_Wuerth_6941xx301002, Connector_BarrelJack:BarrelJack_Wuerth_6941xx301002, F.Cu at (175.7, 106.0)
- added R15: 120 Ohm, Capacitor_SMD:C_0402_1005Metric, F.Cu at (184.5, 94.7)
- added R16: 1K Ohm, Resistor_SMD:R_0402_1005Metric, F.Cu at (183.0, 95.8)
- added R17: 1K Ohm, Resistor_SMD:R_0402_1005Metric, F.Cu at (183.0, 93.5)
- added U5: RS485, Package_SO:SOIC-8_3.9x4.9mm_P1.27mm, F.Cu at (178.5, 94.6)
- F4: value 1.5A 32V -> 1.5A 32V FastBlow
- moved J10 9.96 mm to (185.8, 111.8), turned to 90 degrees
- moved F3 7.78 mm to (186.0, 104.5)
- moved C11 4.90 mm to (169.5, 100.9), turned to 90 degrees
- moved C12 4.47 mm to (165.0, 104.5), turned to 180 degrees
- moved C24 1.00 mm to (151.0, 89.5)
- moved J12 1.00 mm to (165.5, 90.8)
- moved R7 1.00 mm to (163.0, 89.5)
- moved S2 1.00 mm to (155.5, 107.5)
- moved U4 1.00 mm to (157.5, 89.5)
- moved VR2 0.30 mm to (166.6, 113.0)
- renumbered J11 to J12
Connections:
- J8 pad 11: (no net) -> SAM_AD5_PA19_PIN71
- J8 pad 6: RXD1/PA12 -> SAM_PWML7_PC24_PIN135
- J8 pad 8: TDX1/PA13 -> SAM_DAC0_PB15_PIN76
- J8 pad 9: (no net) -> SAM_AD6_PB0_PIN113
- REF** pad 1: RXD0/PA10 -> RXD1/PA12
- REF** pad 1: TXD0/PA11 -> TDX1/PA13
- U1 pad 113: (no net) -> SAM_AD6_PB0_PIN113
- U1 pad 13: (no net) -> SAM_A10_PD0_PIN13
- U1 pad 135: (no net) -> SAM_PWML7_PC24_PIN135
- U1 pad 17: (no net) -> SAM_USART3_RXD_PD4_PIN17
- U1 pad 18: (no net) -> SAM_USART3_TXD_PD5_PIN18
- U1 pad 71: (no net) -> SAM_AD5_PA19_PIN71
- U1 pad 76: (no net) -> SAM_DAC0_PB15_PIN76
Routing:
- net SAM_A10_PD0_PIN13: track 0.00 -> 61.5 mm, vias 0 -> 3
- net SAM_AD5_PA19_PIN71: track 0.00 -> 58.3 mm
- net SAM_USART3_TXD_PD5_PIN18: track 0.00 -> 57.7 mm, vias 0 -> 2
- net SAM_USART3_RXD_PD4_PIN17: track 0.00 -> 54.5 mm, vias 0 -> 2
- net SAM_DAC0_PB15_PIN76: track 0.00 -> 50.8 mm
- net SAM_AD6_PB0_PIN113: track 0.00 -> 42.5 mm
- net GND: track 259.9 -> 291.2 mm, vias 32 -> 40
- net SAM_PWML7_PC24_PIN135: track 0.00 -> 22.1 mm
- net VIN: track 29.4 -> 48.6 mm
- net TDX1/PA13: track 21.8 -> 4.88 mm
- net TWCK0/PA18: track 53.5 -> 69.0 mm
- net RXD1/PA12: track 18.1 -> 3.04 mm
- net MODBUS_B: track 0.00 -> 6.43 mm
- net MODBUS_A: track 0.00 -> 6.40 mm
- net TWD0/PA17: track 33.5 -> 39.3 mm
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Other:
- board text added: "1:GND 2:A1/PWML5/PC22 3:3.3V 4:A2/PWML6/PC23 5:D14/PC16 6:PWML7/PC24 7:D15/PC17 8:DAC0/PB15 9:AD6/PB0 10:TWCK0/PA18 11:AD5/PA19 12:TWD0/PA17"
- board text added: "4pin DipSwitch 1=S-RST 2=E-FLASH 3&4=NC"
- board text added: "5V"
- board text added: "6.5V-24VIN"
- board text added: "MODBUS_A"
- board text added: "MODBUS_B"
- board text added: "SAM 485"
- board text removed: "1:GND 2:A1/PWML5/PC22 3:3.3V 4:A2/PWML6/PC23 5:D14/PC16 6:RXD1/PWML1/PA12 7:D15/PC17 8:TXD1/PWMH2/PA13 9:NC 10:TWCK0/PA18 11:NC 12:TWD0/PA17"
- board text removed: "1=S-RST 2=E-FLASH 3&4=NC"
- board text removed: "6.5V-24V"
