File: RemiRAT.kicad_sch (KiCad schematic)
At the start: 70 parts, among them J1 USB_C_Receptacle_USB2.0_16P, J10 Power In, J11 CANBUS OUT, J11 Power Input Select, J2 ESP32_ARM_JTAG_SWD_10, J3 ESP32 UART0, J4 Micro_SD_Card_Det_Hirose_DM3AT, J5 SAM_ARM_JTAG_SWD_10, J6 SAM UART0, J7 SAM SPI NPCS1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

Commit message: Add files via upload
Parts:
- added C25: 0.1uF 25V, Capacitor_SMD:C_0402_1005Metric, symbol Device:C
- added F5: 1.5A 32V FastBlow, symbol Device:Fuse
- added J12: MODBUS 485 BREAKOUT, symbol Connector:Conn_01x03_Pin
- added J14: 5V OUT, symbol Connector:Conn_01x02_Pin
- added J15: Barrel_Jack, symbol Connector:Barrel_Jack
- added R15: 120 Ohm, Capacitor_SMD:C_0402_1005Metric, symbol Device:R
- added R16, R17: 1K Ohm, Capacitor_SMD:C_0402_1005Metric, symbol Device:R
- added U5: MAX485E, Package_SO:SOIC-8_3.9x4.9mm_P1.27mm, symbol Interface_UART:MAX485E
- renumbered J11 to J12, U5 to U4, U4 to VR2
Connections:
- net +3.3V: now also C25.1, R17.1
- net GND: now also J12.1 (Pin_1), J14.2 (Pin_2), J15.2, R16.2, U5.5 (GND); no longer J4.9 (DET_B), U1.77 (PB16)
- net SAM_AD6_PB0_PIN113: now reaches U1.113 (PB0)
- net SAM_AD6_PB0_PIN113: now also J8.9 (Pin_9)
- net at U1.13 (PD0): now also U5.2 (~{RE}), U5.3 (DE)
- net SAM_PWML7_PC24_PIN135: now reaches U1.135 (PC24)
- net SAM_PWML7_PC24_PIN135: now also J8.6 (Pin_6)
- net SAM_USART3_RXD_PD4_PIN17: now reaches U1.17 (PD4)
- net SAM_USART3_RXD_PD4_PIN17: now also U5.1 (RO)
- net SAM_USART3_TXD_PD5_PIN18: now reaches U1.18 (PD5)
- net SAM_USART3_TXD_PD5_PIN18: now also U5.4 (DI)
- net at R11.2, U2.11 (IO26): now also U1.5 (PA12); no longer U1.3 (PA10)
- net at R9.1, U2.36 (IO22): now also U1.6 (PA13); no longer U1.4 (PA11)
- net SAM_AD5_PA19_PIN71: now reaches U1.71 (PA19)
- net SAM_AD5_PA19_PIN71: now also J8.11 (Pin_11)
- net SAM_DAC0_PB15_PIN76: now reaches U1.76 (PB15)
- net SAM_DAC0_PB15_PIN76: now also J8.8 (Pin_8)
- net at C13.1, J11.1 (Pin_1), VR2.3 (Vout): now also F5.1
- net at F3.1, J10.1 (Pin_1): now also J15.1
- removed net SAM_RXD1_PA12_PIN5: J8.6 (Pin_6), U1.5 (PA12)
- removed net SAM_TXD1_PA13_PIN6: J8.8 (Pin_8), U1.6 (PA13)
- new net: F5.2, J14.1 (Pin_1)
- new net: J12.2 (Pin_2), R15.1, R17.2, U5.6 (A)
- new net: J12.3 (Pin_3), R15.2, R16.1, U5.7 (B)
- new net: C25.2, U5.8 (VCC)
- no-connect marks 104 -> 95
Other:
- note added: "13th July 2025"
- note added: "5VOUT"
- note added: "SAM I2C"
- note added: "SAM RS-485"
- note added: "v01.00"
- note removed: "12th July 2025"
- note removed: "v00.00"
- moved on the sheet: C11, C12, C13, C24, D1, D2, F3, J10, J12, Q1, Q2, R10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
